File: LoRaModule.kicad_sch (KiCad schematic)
At the start: 6 parts, among them J1 Conn_Coaxial, U1 SX127x_Transceiver

Commit message: Add BOM
Parts:
- C2: Manufacturer (none) -> KEMET; PartNumber (none) -> C0603C221J5GACTU
- C7: Manufacturer (none) -> Murata; PartNumber (none) -> GRM188R61C106MA73D
- J1: Manufacturer (none) -> Cinch; PartNumber (none) -> 142-0701-201
Changed lines of the file:
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@@
+      (effects (font (size 1.27 1.27)) hide)
+    )
+    (property "Manufacturer" "Cinch" (id 4) (at 55.88 60.96 0)
+      (effects (font (size 1.27 1.27)) hide)
+    )
+    (property "PartNumber" "142-0701-201" (id 5) (at 55.88 60.96 0)
       (effects (font (size 1.27 1.27)) hide)
     )
@@
     )
     (property "Datasheet" "~" (id 3) (at 133.35 69.85 0)
+      (effects (font (size 1.27 1.27)) hide)
+    )
+    (property "Manufacturer" "Murata" (id 4) (at 133.35 69.85 0)
+      (effects (font (size 1.27 1.27)) hide)
+    )
+    (property "PartNumber" "GRM188R61C106MA73D" (id 5) (at 133.35 69.85 0)
       (effects (font (size 1.27 1.27)) hide)
     )
@@
       (effects (font (size 1.27 1.27)) hide)
     )
+    (property "Manufacturer" "KEMET" (id 4) (at 72.39 60.96 90)
+      (effects (font (size 1.27 1.27)) hide)
+    )
+    (property "PartNumber" "C0603C221J5GACTU" (id 5) (at 72.39 60.96 90)
+      (effects (font (size 1.27 1.27)) hide)
+    )
